File: firmware/Kicad_System_Micro_Lejars_Geslin_Laloux/Kicad_System_Micro_Lejars_Geslin_Laloux.kicad_sch (KiCad schematic)
At the start: 5 parts, among them U1 STM32L021K4Tx

Commit message: Mise à jour
Parts:
- added C2, C3, C4, C5, C6: C_Small, symbol Device:C_Small
Connections:
- net +3.3V: now also C1.1, L1.1, C2.1, C3.1
- net GND: now also C1.2, C2.2, C3.2, C4.2, C5.2
- net at L1.2: now also C4.1, C5.1
- net DAC_nCS: now reaches U1.10 (PA4)
- net SP1_SCK: now reaches U1.11 (PA5)
- net SP1_MOSI: now reaches U1.13 (PA7)
- net LED_STATUS: now reaches U1.18 (PA8)
- net SWDIO: now reaches U1.24 (PA14)
- net SWDCK: now reaches U1.25 (PA15)
- net USUART2_RX: now reaches U1.6 (PA0)
- net ADC_IN1: now reaches U1.7 (PA1)
- net USUART2_TX: now reaches U1.8 (PA2)
- net DAC_nLDAC: now reaches U1.9 (PA3)
Other:
- moved on the sheet: D1, L1, R1
